File: robot-pcb/robot-pcb.sch (KiCad schematic (older format))
At the start: 48 parts, among them J1 Conn_02x03_Counter_Clockwise, J2 Conn_01x05_Female, J3 Conn_02x05_Counter_Clockwise, J4 Conn_01x03_Male, J5 Conn_01x03_Male, J6 Screw_Terminal_01x02, J7 Screw_Terminal_01x02, J8 Screw_Terminal_01x02, J9 Screw_Terminal_01x02, SW1 SW_Push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

Commit message: Remove power switch from pcb
Parts:
- removed SW3: SW_DIP_x01, Button_Switch_SMD:SW_DIP_SPSTx01_Slide_9.78x4.72mm_W8.61mm_P2.54mm, symbol Switch:SW_DIP_x01
- renumbered SW4 to SW3
Connections:
- net +12V: now also J6.2 (Pin_2)
Other:
- moved on the sheet: J6, J9
Changed lines of the file:
@@
 $EndDescr
-$Comp
-L power:GND #PWR0101
-U 1 1 62655056
-P 8950 1400
-F 0 "#PWR0101" H 8950 1150 50  0001 C CNN
-F 1 "GND" H 8955 1227 50  0000 C CNN
-F 2 "" H 8950 1400 50  0001 C CNN
-F 3 "" H 8950 1400 50  0001 C CNN
-	1    8950 1400
-	1    0    0    -1
-$EndComp
 $Comp
 L power:+3V3 #PWR0102
@@
 Text Notes 2150 3200 0    50   ~ 0
 En
-Text Notes 7950 1000 0    50   ~ 0
+Text Notes 8750 900  0    50   ~ 0
 Power
 Text Notes 8250 3650 0    50   ~ 0
@@
 L Connector:Screw_Terminal_01x02 J9
 U 1 1 62656411
-P 9150 1400
-F 0 "J9" H 9250 1300 50  0000 L CNN
-F 1 "Screw_Terminal_01x02" H 9100 1200 50  0000 L CNN
-F 2 "TerminalBlock:TerminalBlock_bornier-2_P5.08mm" H 9150 1400 50  0001 C CNN
-F 3 "~" H 9150 1400 50  0001 C CNN
-	1    9150 1400
+P 9350 1300
+F 0 "J9" H 9450 1200 50  0000 L CNN
+F 1 "Screw_Terminal_01x02" H 9300 1100 50  0000 L CNN
+F 2 "TerminalBlock:TerminalBlock_bornier-2_P5.08mm" H 9350 1300 50  0001 C CNN
+F 3 "~" H 9350 1300 50  0001 C CNN
+	1    9350 1300
 	1    0    0    1
 $EndComp
@@
 L Connector:Screw_Terminal_01x02 J6
 U 1 1 63179D98
-P 8150 1400
-F 0 "J6" H 8068 1075 50  0000 C CNN
-F 1 "Screw_Terminal_01x02" H 8068 1166 50  0000 C CNN
-F 2 "TerminalBlock:TerminalBlock_bornier-2_P5.08mm" H 8150 1400 50  0001 C CNN
-F 3 "~" H 8150 1400 50  0001 C CNN
-	1    8150 1400
+P 8950 1300
+F 0 "J6" H 8868 975 50  0000 C CNN
+F 1 "Screw_Terminal_01x02" H 8868 1066 50  0000 C CNN
+F 2 "TerminalBlock:TerminalBlock_bornier-2_P5.08mm" H 8950 1300 50  0001 C CNN
+F 3 "~" H 8950 1300 50  0001 C CNN
+	1    8950 1300
 	-1   0    0    1
 $EndComp
@@
 L power:GND #PWR0124
 U 1 1 631842F3
-P 8350 1400
-F 0 "#PWR0124" H 8350 1150 50  0001 C CNN
-F 1 "GND" H 8355 1227 50  0000 C CNN
-F 2 "" H 8350 1400 50  0001 C CNN
-F 3 "" H 8350 1400 50  0001 C CNN
-	1    8350 1400
+P 9150 1350
+F 0 "#PWR0124" H 9150 1100 50  0001 C CNN
+F 1 "GND" H 9155 1177 50  0000 C CNN
+F 2 "" H 9150 1350 50  0001 C CNN
+F 3 "" H 9150 1350 50  0001 C CNN
+	1    9150 1350
 	1    0    0    -1
 $EndComp
@@
 L power:+12V #PWR0125
 U 1 1 6318498A
-P 8950 1300
-F 0 "#PWR0125" H 8950 1150 50  0001 C CNN
-F 1 "+12V" H 8965 1473 50  0000 C CNN
-F 2 "" H 8950 1300 50  0001 C CNN
-F 3 "" H 8950 1300 50  0001 C CNN
-	1    8950 1300
+P 9150 1150
+F 0 "#PWR0125" H 9150 1000 50  0001 C CNN
+F 1 "+12V" H 9165 1323 50  0000 C CNN
+F 2 "" H 9150 1150 50  0001 C CNN
+F 3 "" H 9150 1150 50  0001 C CNN
+	1    9150 1150
 	1    0    0    -1
 $EndComp
@@
 Wire Wire Line
 	9750 5000 9700 5000
-$Comp
-L Switch:SW_DIP_x01 SW3
-U 1 1 63210AE4
-P 8650 1300
-F 0 "SW3" H 8650 1567 50  0000 C CNN
-F 1 "SW_DIP_x01" H 8650 1476 50  0000 C CNN
-F 2 "Button_Switch_SMD:SW_DIP_SPSTx01_Slide_9.78x4.72mm_W8.61mm_P2.54mm" H 8650 1300 50  0001 C CNN
-F 3 "~" H 8650 1300 50  0001 C CNN
-	1    8650 1300
-	1    0    0    -1
-$EndComp
 Connection ~ 8800 4500
 Connection ~ 8800 4900
-Connection ~ 8950 1300
 $Comp
 L Device:R R11
@@
 	4000 1350 4000 1600
 $Comp
-L Switch:SW_DPST_x2 SW4
+L Switch:SW_DPST_x2 SW3
 U 1 1 6327B921
 P 4600 1500
-F 0 "SW4" H 4850 1700 50  0000 C CNN
+F 0 "SW3" H 4850 1700 50  0000 C CNN
 F 1 "SW_DPST_x2" H 4900 1600 50  0000 C CNN
 F 2 "Connector_PinHeader_2.54mm:PinHeader_1x02_P2.54mm_Vertical" H 4600 1500 50  0001 C CNN
@@
 Wire Wire Line
 	4800 1550 4800 1500
+Connection ~ 9150 1200
+Wire Wire Line
+	9150 1150 9150 1200
+Wire Wire Line
+	9150 1300 9150 1350
+Connection ~ 9150 1300
 $EndSCHEMATC

Commit message: Finish pcb v1.0
Parts:
- removed J1: Conn_02x03_Counter_Clockwise, Connector_PinHeader_1.27mm:PinHeader_2x03_P1.27mm_Vertical_SMD, symbol Connector_Generic:Conn_02x03_Counter_Clockwise
- removed J3: Conn_02x05_Counter_Clockwise, Connector_PinHeader_1.27mm:PinHeader_2x05_P1.27mm_Vertical_SMD, symbol Connector_Generic:Conn_02x05_Counter_Clockwise
- added J1: Conn_02x03_Odd_Even, Connector_PinHeader_1.27mm:PinHeader_2x03_P1.27mm_Vertical_SMD, symbol Connector_Generic:Conn_02x03_Odd_Even
- added J3: Conn_02x05_Odd_Even, Connector_PinHeader_1.27mm:PinHeader_2x05_P1.27mm_Vertical_SMD, symbol Connector_Generic:Conn_02x05_Odd_Even
- R10, R7: value 330 -> 68
- SW1, SW2: footprint Button_Switch_SMD:SW_Push_SPST_NO_Alps_SKRK -> robot-pcb_custom:wurth_tactile_sw
Connections:
- net +3V3: now also J1.2 (Pin_2), J3.1 (Pin_1)
- net EN: now also J1.1 (Pin_1)
- net GND: now also J1.4 (Pin_4), J3.3 (Pin_3), J3.5 (Pin_5), J3.7 (Pin_7), J3.9 (Pin_9)
- net IO0: now also J1.6 (Pin_6)
- net RX0D: now also J1.5 (Pin_5)
- net TX0D: now also J1.3 (Pin_3)
- net at R5.1: now also J3.6 (Pin_6)
- net at R3.1: now also J3.2 (Pin_2)
- net at R4.1: now also J3.4 (Pin_4)
- net at R6.1: now also J3.8 (Pin_8)
Changed lines of the file:
@@
 F 0 "SW2" H 3000 3600 50  0000 L CNN
 F 1 "SW_Push" H 3000 3500 50  0000 L CNN
-F 2 "Button_Switch_SMD:SW_Push_SPST_NO_Alps_SKRK" H 3150 3500 50  0001 C CNN
+F 2 "robot-pcb_custom:wurth_tactile_sw" H 3150 3500 50  0001 C CNN
 F 3 "~" H 3150 3500 50  0001 C CNN
 	1    3150 3300
@@
 F 0 "SW1" H 2650 3600 50  0000 R CNN
 F 1 "SW_Push" H 2650 3500 50  0000 R CNN
-F 2 "Button_Switch_SMD:SW_Push_SPST_NO_Alps_SKRK" H 2500 3500 50  0001 C CNN
+F 2 "robot-pcb_custom:wurth_tactile_sw" H 2500 3500 50  0001 C CNN
 F 3 "~" H 2500 3500 50  0001 C CNN
 	1    2500 3300
@@
 	1    5700 6900
 	0    -1   -1   0
-$EndComp
-$Comp
-L Connector_Generic:Conn_02x05_Counter_Clockwise J3
-U 1 1 6271D303
-P 5250 6800
-F 0 "J3" H 5300 7217 50  0000 C CNN
-F 1 "Conn_02x05_Counter_Clockwise" H 5300 7126 50  0000 C CNN
-F 2 "Connector_PinHeader_1.27mm:PinHeader_2x05_P1.27mm_Vertical_SMD" H 5250 6800 50  0001 C CNN
-F 3 "~" H 5250 6800 50  0001 C CNN
-	1    5250 6800
-	1    0    0    -1
 $EndComp
 $Comp
@@
 Text GLabel 1750 6700 0    50   Input ~ 0
 EN
-$Comp
-L Connector_Generic:Conn_02x03_Counter_Clockwise J1
-U 1 1 631362EE
-P 1950 6800
-F 0 "J1" H 2000 7117 50  0000 C CNN
-F 1 "Conn_02x03_Counter_Clockwise" H 2000 7026 50  0000 C CNN
-F 2 "Connector_PinHeader_1.27mm:PinHeader_2x03_P1.27mm_Vertical_SMD" H 1950 6800 50  0001 C CNN
-F 3 "~" H 1950 6800 50  0001 C CNN
-	1    1950 6800
-	1    0    0    -1
-$EndComp
 Text Notes 1050 6400 0    50   ~ 0
 Programming interface
@@
 P 9350 2300
 F 0 "R7" V 9450 2300 50  0000 C CNN
-F 1 "330" V 9550 2300 50  0000 C CNN
+F 1 "68" V 9550 2300 50  0000 C CNN
 F 2 "Resistor_SMD:R_0603_1608Metric_Pad0.98x0.95mm_HandSolder" V 9280 2300 50  0001 C CNN
 F 3 "~" H 9350 2300 50  0001 C CNN
@@
 U 1 1 62656411
 P 9350 1300
-F 0 "J9" H 9450 1200 50  0000 L CNN
+F 0 "J9" H 9300 1400 50  0000 L CNN
 F 1 "Screw_Terminal_01x02" H 9300 1100 50  0000 L CNN
 F 2 "TerminalBlock:TerminalBlock_bornier-2_P5.08mm" H 9350 1300 50  0001 C CNN
@@
 U 1 1 63179D98
 P 8950 1300
-F 0 "J6" H 8868 975 50  0000 C CNN
+F 0 "J6" H 8950 1400 50  0000 C CNN
 F 1 "Screw_Terminal_01x02" H 8868 1066 50  0000 C CNN
 F 2 "TerminalBlock:TerminalBlock_bornier-2_P5.08mm" H 8950 1300 50  0001 C CNN
@@
 P 3700 3600
 F 0 "R10" H 3770 3646 50  0000 L CNN
-F 1 "330" H 3770 3555 50  0000 L CNN
+F 1 "68" H 3770 3555 50  0000 L CNN
 F 2 "Resistor_SMD:R_0603_1608Metric_Pad0.98x0.95mm_HandSolder" V 3630 3600 50  0001 C CNN
 F 3 "~" H 3700 3600 50  0001 C CNN
@@
 	9150 1300 9150 1350
 Connection ~ 9150 1300
+$Comp
+L Connector_Generic:Conn_02x05_Odd_Even J3
+U 1 1 632CCE3A
+P 5250 6800
+F 0 "J3" H 5300 7217 50  0000 C CNN
+F 1 "Conn_02x05_Odd_Even" H 5300 7126 50  0000 C CNN
+F 2 "Connector_PinHeader_1.27mm:PinHeader_2x05_P1.27mm_Vertical_SMD" H 5250 6800 50  0001 C CNN
+F 3 "~" H 5250 6800 50  0001 C CNN
+	1    5250 6800
+	1    0    0    -1
+$EndComp
+$Comp
+L Connector_Generic:Conn_02x03_Odd_Even J1
+U 1 1 632E355A
+P 1950 6800
+F 0 "J1" H 2000 7117 50  0000 C CNN
+F 1 "Conn_02x03_Odd_Even" H 2000 7026 50  0000 C CNN
+F 2 "Connector_PinHeader_1.27mm:PinHeader_2x03_P1.27mm_Vertical_SMD" H 1950 6800 50  0001 C CNN
+F 3 "~" H 1950 6800 50  0001 C CNN
+	1    1950 6800
+	1    0    0    -1
+$EndComp
 $EndSCHEMATC
