File: robot-pcb/robot-pcb.kicad_pcb (KiCad board)
At the start: 2 copper layers, 59.7 x 47 mm, 51 parts, among them J1 Conn_02x03_Counter_Clockwise, J2 Conn_01x05_Female, J3 Conn_02x05_Counter_Clockwise, J4 Conn_01x03_Male, J5 Conn_01x03_Male, J6 Screw_Terminal_01x02, J7 Screw_Terminal_01x02, J8 Screw_Terminal_01x02, J9 Screw_Terminal_01x02, SW1 SW_Push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

Commit message: Remove power switch from pcb
Parts:
- removed the SW3 at (123.8, 57.8)
- renumbered SW4 to SW3
Connections:
- J6 pad 2: Net-(J6-Pad2) -> +12V
- U2 pad 4: (no net) -> +3V3
Routing:
- net Net-(J6-Pad2): track 6.75 -> 0.00 mm
- net +12V: track 70.4 -> 74.7 mm
- net nSLEEP: track 86.7 -> 90.1 mm, vias 1 -> 2
- net nFAULT: track 74.0 -> 76.1 mm
- net GND: track 26.1 -> 27.5 mm, vias 17 -> 16
- net +3V3: track 132.3 -> 133.4 mm
Other:
- board size 59.7 x 47 mm -> 61.6 x 47 mm
- board text added: "+12V"
- board text added: "12V in/out"
- board text added: "GND"
- board text added: "Motor A"
- board text added: "Motor B"

Commit message: Finish pcb v1.0
Parts:
- added G***: LOGO, robot-pcb_custom:rupert_bitmap_art, F.Cu at (122.7, 58.8)
- J1: value Conn_02x03_Counter_Clockwise -> Conn_02x03_Odd_Even
- J3: value Conn_02x05_Counter_Clockwise -> Conn_02x05_Odd_Even
- R10, R7: value 330 -> 68
- SW1, SW2: footprint Button_Switch_SMD:SW_Push_SPST_NO_Alps_SKRK -> robot-pcb_custom:wurth_tactile_sw
- moved C4 1.08 mm to (99.1, 94.0)
- moved SW1 1.08 mm to (102.2, 94.0)
- moved SW2 1.08 mm to (102.2, 85.1)
- moved C5 1.06 mm to (99.1, 85.1)
- moved J3 0.13 mm to (92.1, 85.9), turned to 90 degrees
- moved J1 0.13 mm to (92.1, 94.7)
Connections:
- J1 pad 2: TX0D -> +3V3
- J1 pad 3: RX0D -> TX0D
- J1 pad 4: IO0 -> GND
- J1 pad 5: GND -> RX0D
- J1 pad 6: +3V3 -> IO0
- J3 pad 2: GND -> Net-(J3-Pad2)
- J3 pad 4: GND -> Net-(J3-Pad4)
- J3 pad 6: (no net) -> Net-(J3-Pad6)
- J3 pad 7: Net-(J3-Pad7) -> GND
- J3 pad 9: Net-(J3-Pad9) -> GND
- R3 pad 1: Net-(J3-Pad10) -> Net-(J3-Pad2)
- R4 pad 1: Net-(J3-Pad9) -> Net-(J3-Pad4)
- R5 pad 1: Net-(J3-Pad8) -> Net-(J3-Pad6)
- R6 pad 1: Net-(J3-Pad7) -> Net-(J3-Pad8)
Routing:
- net Net-(J3-Pad4): track 0.00 -> 16.3 mm, vias 0 -> 2
- net Net-(J3-Pad6): track 0.00 -> 10.1 mm
- net Net-(J3-Pad7): track 9.59 -> 0.00 mm
- net Net-(J3-Pad10): track 8.38 -> 0.00 mm
- net Net-(J3-Pad8): track 12.1 -> 4.81 mm
- net GND: track 27.5 -> 20.3 mm, vias 16 -> 18
- net TX0D: track 64.2 -> 57.9 mm
- net Net-(J3-Pad9): track 5.59 -> 0.00 mm
- net Net-(J3-Pad2): track 0.00 -> 4.01 mm
- net +3V3: track 133.4 -> 137.2 mm, vias 2 -> 1
- net RX0D: track 64.9 -> 62.9 mm
- net IO0: track 26.4 -> 24.6 mm
- net EN: track 58.2 -> 57.5 mm
Other:
- board text added: "+"
- board text added: "En"
- board text added: "IO0"
- board text added: "Rupert brain pcb v1.0"

Commit message: Update robot pcb holder and update kicad version
Other:
- net class Default removed
